Commit message: Minor tweaks

File: packages/leap-motion-controller/urdf/hands_fix.urdf (robot description, URDF)
Before this commit: robot leap_hands, 3 links, 2 joints
Links:
- link leap_left_hand: geometry visual mesh filename=package://leap_motion_controller/urdf/meshes/hand.stl scale=-0.001 0.001 0.001
- link leap_right_hand: geometry visual mesh filename=package://leap_motion_controller/urdf/meshes/hand.stl scale=0.001 0.001 0.001
