Commit message: Added visualisation for sensor max range

File: leap_motion_controller/urdf/hands_fix.urdf (robot description, URDF)
Before this commit: robot leap_hands, 3 links, 2 joints
Links:
- link leap_base_link: geometry visual box size=0.7 0.7 0.7

Commit message: minor

File: leap_motion_controller/urdf/hands_fix.urdf (robot description, URDF)
Before this commit: robot leap_hands, 3 links, 2 joints
Links:
- link leap_base_link: geometry visual box size=0.7 0.8 0.7
